File: TempSense.kicad_pcb (KiCad board)
At the start: 2 copper layers, 40 x 22.1 mm, 36 parts, among them J1 Conn_01x02_Pin, P1 USB_C_Plug_USB2.0, SW1 SW_Push, SW2 SW_Push, U1 MCP73831-2-OT, U2 BME680, U3 AP2112K-3.3, U4 ESP32-C6-MINI-1

Commit message: stuffs
Parts:
- added C14: 100nF, Capacitor_SMD:C_0402_1005Metric, F.Cu at (170.2, 85.3)
- added R10: 10k, Resistor_SMD:R_0402_1005Metric, F.Cu at (172.8, 85.8)
- C13: value 1uF -> 10uF
- moved SW1 11.1 mm to (179.5, 72.5), turned to -90 degrees
- moved C13 10.6 mm to (175.5, 74.7)
- moved J1 7.17 mm to (163.7, 89.2)
- moved R9 5.09 mm to (177.1, 74.3)
- moved C7 4.09 mm to (160.4, 84.2), turned to 0 degrees
- moved D6 3.37 mm to (164.1, 86.4)
- moved SW2 2.96 mm to (170.8, 88.0)
- moved C6 2.83 mm to (182.8, 74.5)
- moved U4 2.59 mm to (179.8, 82.5)
- moved R5 2.46 mm to (172.9, 81.6)
- moved R6 2.44 mm to (172.9, 82.7)
- moved U3 2.36 mm to (158.4, 86.5)
- moved C5 2.27 mm to (167.9, 83.3)
Connections:
- C13 pad 1: Net-(C13-Pad1) -> /EN
- SW1 pad 1: Net-(C13-Pad1) -> GND
Routing:
- net GND: track 33.7 -> 52.9 mm, vias 17 -> 22
- net +3V3: track 109.4 -> 102.5 mm
- net /LED: track 7.77 -> 13.0 mm
- net /SDA-BME680: track 27.2 -> 31.8 mm
- net Net-(D6-K): track 11.3 -> 9.38 mm
- net /boot: track 8.14 -> 9.49 mm
- net Net-(C13-Pad1): track 1.31 -> 0.00 mm
- net /EN: track 7.35 -> 6.20 mm
- net /SCL-BME680: track 30.3 -> 31.4 mm
- net Net-(P1-D+): track 19.4 -> 20.2 mm
- net Net-(P1-D-): track 20.0 -> 20.8 mm, vias 0 -> 2
- net /STAT: track 20.4 -> 21.1 mm, vias 2 -> 0
Other:
- outline, holes or cut-outs redrawn
- board text added: "(kaze)"
- board text added: "If you're seeing this, kudos!"
- board text added: "かぜ"
- board text removed: "BME680 goes here"
