File: TempSense.kicad_sch (KiCad schematic)
At the start: 36 parts, among them J1 Conn_01x02_Pin, P1 USB_C_Plug_USB2.0, SW1 SW_Push, SW2 SW_Push, U1 MCP73831-2-OT, U2 BME680, U3 AP2112K-3.3, U4 ESP32-C6-MINI-1

Commit message: stuffs
Parts:
- added C14: 100nF, Capacitor_SMD:C_0402_1005Metric, symbol Device:C
- added R10: 10k, Resistor_SMD:R_0402_1005Metric, symbol Device:R
- added TP1, TP2, TP3, TP4, TP5: TestPoint, symbol Connector:TestPoint
- C13: value 1uF -> 10uF
Connections:
- net +3V3: now also R10.1
- net EN: now also C13.1
- net GND: now also SW1.1, C14.2
- net boot: now also C14.1, R10.2
- net IO18: now reaches U4.24 (IO18)
- net IO18: now also TP1.1
- net IO19: now reaches U4.25 (IO19)
- net IO19: now also TP2.1
- net IO20: now reaches U4.26 (IO20)
- net IO20: now also TP3.1
- net IO21: now reaches U4.27 (IO21)
- net IO21: now also TP4.1
- net IO22: now reaches U4.28 (IO22)
- net IO22: now also TP5.1
- net BAT+ renamed +BATT
Other:
- moved on the sheet: C13, R9, SW1, SW2
