File: kaze.kicad_pcb (KiCad board)
At the start: 2 copper layers, 40 x 22.1 mm, 48 parts, among them J1 Conn_01x02_Pin, P1 USB_C_Plug_USB2.0, SW1 SW_Push, SW2 SW_Push, U1 MCP73831-2-OT, U2 BME680, U3 AP2112K-3.3, U4 ESP32-C6-MINI-1, U5 TSL25911FN, U6 SGP40-D-R4

Commit message: v1?
Parts:
- added IO2: TestPoint, TestPoint:TestPoint_Pad_D3.0mm, B.Cu at (183.4, 70.9)
- added IO3: TestPoint, TestPoint:TestPoint_Pad_D3.0mm, B.Cu at (179.0, 70.9)
Connections:
- U4 pad 24: /IO18 -> unconnected-(U4-IO18-Pad24)
- U4 pad 25: /IO19 -> unconnected-(U4-IO19-Pad25)
- U4 pad 26: /IO20 -> unconnected-(U4-IO20-Pad26)
- U4 pad 27: /IO21 -> unconnected-(U4-IO21-Pad27)
- U4 pad 28: /IO22 -> unconnected-(U4-IO22-Pad28)
- U4 pad 5: unconnected-(U4-IO2-Pad5) -> /IO2
- U4 pad 6: unconnected-(U4-IO3-Pad6) -> /IO3
Routing:
- net /IO2: track 0.00 -> 8.79 mm, vias 0 -> 1
- net /IO3: track 0.00 -> 6.81 mm, vias 0 -> 1
- net GND: track 59.6 -> 60.9 mm, vias 28 -> 31
