File: kaze.kicad_sch (KiCad schematic)
At the start: 51 parts, among them J1 Conn_01x02_Pin, P1 USB_C_Plug_USB2.0, SW1 SW_Push, SW2 SW_Push, U1 MCP73831-2-OT, U2 BME680, U3 AP2112K-3.3, U4 ESP32-C6-MINI-1, U5 TSL25911FN, U6 SGP40-D-R4

Commit message: v1?
Parts:
- removed TP2, TP4, TP5: TestPoint, symbol Connector:TestPoint
- TP1: footprint (none) -> TestPoint:TestPoint_Pad_D3.0mm
- TP2: renamed from TP3; footprint (none) -> TestPoint:TestPoint_Pad_D3.0mm
Connections:
- net IO2: now reaches U4.5 (IO2)
- net IO2: now also TP1.1
- net IO3: now reaches U4.6 (IO3)
- net IO3: now also TP2.1
- net IO18: no longer names the net of U4.24 (IO18)
- net IO18: no longer TP1.1
- net IO19: no longer names the net of U4.25 (IO19)
- net IO20: no longer names the net of U4.26 (IO20)
- net IO20: no longer TP2.1
- net IO21: no longer names the net of U4.27 (IO21)
- net IO22: no longer names the net of U4.28 (IO22)
- no-connect marks 11 -> 14
